File: Hardware/Interactive_SparkFun_Badge.brd (EAGLE design)
At the start: 88.9 x 63.5 mm, 30 parts, among them J1 AVR_SPI_PRG_6PTH, U1 ATMEGA328P

Commit message: Adding Rome MF back silk
Parts:
- U$2: value NY_FAIRE_BACK -> ROME_FAIRE_BACK; device Local Library:NY_BACK -> Local Library:ROME_BACK
- moved U$2 4.58 mm to (-1.27, -3.81)
Changed lines of the file:
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@@
 <layer number="47" name="Measures" color="7" fill="1" visible="no" active="yes"/>
 <layer number="48" name="Document" color="7" fill="1" visible="no" active="yes"/>
-<layer number="49" name="Reference" color="7" fill="1" visible="yes" active="yes"/>
+<layer number="49" name="Reference" color="7" fill="1" visible="no" active="yes"/>
 <layer number="50" name="dxf" color="7" fill="1" visible="no" active="no"/>
 <layer number="51" name="tDocu" color="6" fill="1" visible="yes" active="yes"/>
@@
 </element>
 <element name="U$4" library="Local Library" package="FAIRE_GAME_SILK" value="FAIRE_GAME_SILK" x="-0.635" y="-0.762"/>
-<element name="U$2" library="Local Library" package="NY_BACK" value="NY_FAIRE_BACK" x="1.27" y="0"/>
+<element name="U$2" library="Local Library" package="ROME_BACK" value="ROME_FAIRE_BACK" x="-1.27" y="-3.81"/>
 </elements>
 <signals>
