File: Hardware/Interactive_SparkFun_Badge.brd (EAGLE design)
At the start: 88.9 x 63.5 mm, 30 parts, among them J1 AVR_SPI_PRG_6PTH, U1 ATMEGA328P

Commit message: Switching to Schottky diode
Parts:
- D3, D4: value DIODE-ZENER3.3V -> PMEG4005EJ
Changed lines of the file:
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@@
 <element name="J1" library="SparkFun-Connectors" package="2X3" value="AVR_SPI_PRG_6PTH" x="85.09" y="40.64" rot="R270"/>
 <element name="U$3" library="ML8511" package="INITIALS" value="ALPHABET" x="60.325" y="43.815" rot="R180"/>
-<element name="D3" library="SparkFun-DiscreteSemi" package="SOD-323" value="DIODE-ZENER3.3V" x="9.525" y="22.86" rot="R180">
-<attribute name="PROD_ID" value="DIO-11284" x="9.525" y="22.86" size="1.778" layer="27" font="vector" ratio="15" rot="R180" display="off"/>
-<attribute name="VALUE" value="3.3V" x="9.525" y="22.86" size="1.778" layer="27" rot="R180" display="off"/>
+<element name="D3" library="SparkFun-DiscreteSemi" package="SOD-323" value="PMEG4005EJ" x="9.525" y="22.86" rot="R180">
+<attribute name="PROD_ID" value="DIO-10955" x="9.525" y="22.86" size="1.778" layer="27" font="vector" ratio="15" rot="R180" display="off"/>
+<attribute name="VALUE" value="PMEG4005EJ" x="9.525" y="22.86" size="1.778" layer="27" rot="R180" display="off"/>
 </element>
-<element name="D4" library="SparkFun-DiscreteSemi" package="SOD-323" value="DIODE-ZENER3.3V" x="78.105" y="3.175" rot="R90">
-<attribute name="PROD_ID" value="DIO-11284" x="78.105" y="3.175" size="1.778" layer="27" font="vector" ratio="15" rot="R90" display="off"/>
-<attribute name="VALUE" value="3.3V" x="78.105" y="3.175" size="1.778" layer="27" rot="R90" display="off"/>
+<element name="D4" library="SparkFun-DiscreteSemi" package="SOD-323" value="PMEG4005EJ" x="78.105" y="3.175" rot="R90">
+<attribute name="PROD_ID" value="DIO-10955" x="78.105" y="3.175" size="1.778" layer="27" font="vector" ratio="15" rot="R90" display="off"/>
+<attribute name="VALUE" value="PMEG4005EJ" x="78.105" y="3.175" size="1.778" layer="27" rot="R90" display="off"/>
 </element>
 <element name="C1" library="SparkFun-Capacitors" package="0603-CAP" value="0.1uF" x="9.525" y="30.48">
