File: Hardware/Interactive_SparkFun_Badge.sch (EAGLE design)
At the start: 30 parts, among them J1 AVR_SPI_PRG_6PTH, U1 ATMEGA328P

Commit message: Fixing version number to v10
Other:
- note added: "v10"
- note removed: "v01"
Changed lines of the file:
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@@
 <sheet>
 <plain>
-<text x="238.76" y="7.62" size="2.54" layer="94">v01</text>
+<text x="238.76" y="7.62" size="2.54" layer="94">v10</text>
 <text x="166.116" y="11.43" size="2.54" layer="94">Toni Klopfenstein</text>
 <wire x1="0" y1="114.3" x2="58.42" y2="114.3" width="0" layer="94" style="shortdash"/>
